Commit message: tiene patas.

File: champ/champ_description/urdf/asus_camera.urdf.xacro (robot description, xacro)
@@ -21,5 +21,5 @@
           <origin xyz="0 0 0" rpy="0 0 0" />
           <geometry>
-            <mesh filename="file://$(find champ_description)/meshes/asus_camera_simple.dae"/>
+            <mesh filename="package://champ_description/meshes/asus_camera_simple.dae"/>
           </geometry>
         </visual>
@@ -35,5 +35,5 @@
           <origin xyz="0 0 0" rpy="0 0 0" />
           <geometry>
-            <mesh filename="file://$(find champ_description)/meshes/asus_camera_simple.dae"/>
+            <mesh filename="package://champ_description/meshes/asus_camera_simple.dae"/>
           </geometry>
         </collision>

File: champ/champ_description/urdf/champ.urdf.xacro (robot description, xacro)
@@ -13,5 +13,5 @@
             <origin xyz="0 0 0" rpy="0 0 0" />
             <geometry>
-                <mesh filename="file://$(find champ_description)/meshes/base_simple.stl" scale="0.001 0.001 0.001" />
+                <mesh filename="package://champ_description/meshes/base_simple.stl" scale="0.001 0.001 0.001" />
             </geometry>
             <material name="black" />
@@ -64,4 +64,6 @@
     </plugin>
     </gazebo>
+    <!-- Comentado porque go2_description ya tiene su propio plugin gazebo_ros2_control -->
+    <!--
     <gazebo>
         <plugin filename="libgazebo_ros2_control.so" name="gazebo_ros2_control">
@@ -69,3 +71,4 @@
       </plugin>
     </gazebo>
+    -->
 </robot>

File: champ/champ_description/urdf/hokuyo_utm30lx.urdf.xacro (robot description, xacro)
@@ -17,5 +17,5 @@
           <origin xyz="0 0 0" rpy="0 0 0" />
           <geometry>
-          <mesh filename="file://$(find champ_description)/meshes/hokuyo_utm_30lx$(optenv TEST_SELF_FILTER).dae"/>
+          <mesh filename="package://champ_description/meshes/hokuyo_utm_30lx$(optenv TEST_SELF_FILTER).dae"/>
         </geometry>
         </visual>

File: champ/champ_description/urdf/properties.urdf.xacro (robot description, xacro)
@@ -6,20 +6,20 @@
     <xacro:property name="upper_leg_to_lower_leg_distance" value="0.141" />
     <xacro:property name="lower_leg_to_foot_distance" value="0.141" />
-    <xacro:property name="hip_mesh_path" value="file://$(find champ_description)/meshes/hip.stl" />
+    <xacro:property name="hip_mesh_path" value="package://champ_description/meshes/hip.stl" />
     <xacro:property name="hip_mass" value="0.250" />
     <xacro:property name="hip_x_length" value="0.112" />
     <xacro:property name="hip_y_length" value="0.08" />
     <xacro:property name="hip_z_length" value="0.130" />
-    <xacro:property name="upper_leg_mesh_path" value="file://$(find champ_description)/meshes/upper_leg_simple.stl" />
+    <xacro:property name="upper_leg_mesh_path" value="package://champ_description/meshes/upper_leg_simple.stl" />
     <xacro:property name="upper_leg_mass" value="0.125" />
     <xacro:property name="upper_leg_x_length" value="0.05" />
     <xacro:property name="upper_leg_y_length" value="0.03" />
     <xacro:property name="upper_leg_z_length" value="0.1905" />
-    <xacro:property name="lower_leg_mesh_path" value="file://$(find champ_description)/meshes/lower_leg_simple.stl" />
+    <xacro:property name="lower_leg_mesh_path" value="package://champ_description/meshes/lower_leg_simple.stl" />
     <xacro:property name="lower_leg_mass" value="0.125" />
     <xacro:property name="lower_leg_x_length" value="0.039" />
     <xacro:property name="lower_leg_y_length" value="0.022" />
     <xacro:property name="lower_leg_z_length" value="0.156" />
-    <xacro:property name="base_mesh_path" value="file://$(find champ_description)/meshes/base_simple.stl" />
+    <xacro:property name="base_mesh_path" value="package://champ_description/meshes/base_simple.stl" />
     <xacro:property name="base_mass" value="2.0" />
     <xacro:property name="base_x_length" value="0.5" />
